Commit message: Sync with Jetson

File: src/backend/description/robot.urdf.xacro (robot description, xacro)
@@ -51,5 +51,5 @@
     </link>
     <xacro:include filename="robot_actuator.xacro"   />
-    <xacro:include filename="robot_imu.xacro"       />
+    <!-- xacro:include filename="robot_imu.xacro"       / -->
     <xacro:include filename="robot_depth.xacro"     />
     <xacro:include filename="robot_gazebo.xacro" />

File: src/backend/description/robot_imu.xacro (robot description, xacro)
@@ -2,9 +2,10 @@
 <robot xmlns:xacro="http://www.ros.org/wiki/xacro">
     <xacro:include filename="robot_properties.xacro"/>
+    <!-- Sim IMU is attached to the front facing depth camera, similar to real bot -->
     <link name="imu_link">
         <origin xyz="0 0 0" rpy="0 0 0"/>
     </link>
     <joint name="imu_joint" type="fixed">
-        <parent link="base_link"/>
+        <parent link="depth_link"/>
         <child link="imu_link"/>
         <origin xyz="${imu_x} ${imu_y} ${imu_z}" rpy="0 0 0"/>
@@ -28,5 +29,5 @@
         <rpyOffset>0 0 0</rpyOffset>
         <frameName>imu_link</frameName>
-        <initialOrientationAsReference>false</initialOrientationAsReference>
+        <initialOrientationAsReference>true</initialOrientationAsReference>
       </plugin>
       <pose>0 0 0 0 0 0</pose>
