Commit message: Added gz_worlds Fixed paths in launch files not being machine-agnostic Reorganized some files in frontend and backend Added clean install script Added more documentation

File: src/backend/description/robot_servo.xacro (robot description, xacro)
@@ -3,30 +3,99 @@
     <xacro:include filename="robot_properties.xacro"/>
     <xacro:include filename="robot_inertia.xacro" />
+    <link name="actuator_base_link">
+        <origin xyz="0 0 0" />
+        <visual>
+            <origin xyz="0 0 -${actuator_height / 2}" />
+            <geometry>
+                <box size="${actuator_size} ${actuator_size} ${actuator_height}"/>
+            </geometry>
+            <material name="grey" />
+        </visual>
+        <collision>
+            <origin xyz="0 0 -${actuator_height / 2}" />
+            <geometry>
+                <box size="${actuator_size} ${actuator_size} ${actuator_height}"/>
+            </geometry>
+        </collision>
+        <xacro:inertial_box mass="6.0" x="${actuator_size}" y="${actuator_size}" z="${actuator_height}"/>
+    </link>
+    <joint name="actuator_base_joint" type="fixed" >
+        <parent link="base_link" />
+        <child link="actuator_base_link" />
+        <origin xyz="0 ${(base_width + actuator_size) / 2} ${actuator_height}" rpy="0 0 0" />
+    </joint>
     <link name="servo_link">
         <origin xyz="0 0 0" rpy="0 0 0"/>
         <visual>
-            <origin xyz="0 0 0.05" rpy="0 0 0"/>
+            <origin xyz="0 0 0" rpy="0 0 0"/>
             <geometry>
                 <!-- cylinder length="0.1" radius="0.1" / -->
-                <box size="0.1 0.1 0.1"/>
+                <box size="${actuator_size} ${actuator_size} ${actuator_size}"/>
             </geometry>
         </visual>
         <collision>
-            <origin xyz="0 0.05 0" rpy="0 0 0"/>
+            <origin xyz="0 0 0" rpy="0 0 0"/>
             <geometry>
                 <!-- cylinder length="0.1" radius="0.1" / -->
-                <box size="0.1 0.1 0.1"/>
+                <box size="${actuator_size} ${actuator_size} ${actuator_size}"/>
             </geometry>
         </collision>
         <xacro:inertial_cylinder mass="1.0" length="0.1" radius="0.1" >
-            <origin xyz="0 0 0.05" rpy="0 0 0"/>
+            <origin xyz="0 0 0" rpy="0 0 0"/>
         </xacro:inertial_cylinder>
     </link>
     <joint name="servo_joint" type="continuous">
-        <parent link="base_link" />
+        <parent link="actuator_base_link" />
         <child link="servo_link" />
-        <origin rpy="0 0 0" xyz="0 0 ${base_height / 2}" />
+        <origin rpy="0 0 0.015" xyz="0 0 ${base_height / 2}" />
         <axis rpy="0 0 0" xyz="0 0 1"/>
         <limit effort="100" velocity="100" />
     </joint>
+ <link name="rgb_link">
+        <origin xyz="0 0 0.015" rpy="0 0 0"/>
+        <visual>
+            <geometry>
+                <box size="0.03 0.03 0.03"/>
+            </geometry>
+        </visual>
+        <material name="blue" />
+    </link>
+    <joint name="rgb_joint" type="fixed">
+        <parent link="servo_link" />
+        <child link="rgb_link" />
+        <origin xyz="0 0 0.045" rpy="0 0 0"/>
+    </joint>
+    <!-- This is for transformations between image frame and world frame -->
+    <link name="rgb_link_optical"></link>
+    <joint name="rgb_optical_joint" type="fixed">
+        <parent link="rgb_link" />
+        <child link="rgb_link_optical" />
+        <origin xyz="0 0 0" rpy="${-pi/2} 0 ${-pi/2}"/>
+    </joint>
+    <gazebo reference="rgb_link">
+        <material>Gazebo/Blue</material>
+        <sensor name="rgb" type="camera">
+            <pose> 0 0 0 0 0 0 </pose>
+            <visualize>true</visualize>
+            <update_rate>10</update_rate>
+            <camera>
+                <horizontal_fov>1.57079632679</horizontal_fov>
+                <image>
+                    <format>R8G8B8</format>
+                    <width>640</width>
+                    <height>480</height>
+                </image>
+                <clip>
+                    <near>0.01</near>
+                    <far>11.0</far>
+                </clip>
+            </camera>
+            <plugin name="rgb_controller" filename="libgazebo_ros_camera.so">
+                <frame_name>rgb_link_optical</frame_name>
+                <ros>
+                    <namespace>camera</namespace>
+                </ros>
+            </plugin>
+        </sensor>
+    </gazebo>
 </robot>
